Commit message: Modified Openrve and Gazebo environment Tested Gazebo simulation with tote and shelf

File: stowing/src/stowing_driver/urdf/apc_shelf.urdf.xacro (robot description, xacro)
@@ -14,5 +14,5 @@
         <origin xyz="${X} ${Y} ${Z}" rpy="${roll} ${pitch} ${yaw}"/>
         <geometry>
-           <mesh filename="package://stowing_driver/scripts/pod_lowres.stl" />
+           <mesh filename="package://stowing_driver/meshes/pod_lowres.stl" />
         </geometry>
       </visual>
@@ -20,5 +20,5 @@
         <origin xyz="${X} ${Y} ${Z}" rpy="${roll} ${pitch} ${yaw}"/>
         <geometry>
-           <mesh filename="package://stowing_driver/scripts/pod_lowres.stl" />
+           <mesh filename="package://stowing_driver/meshes/pod_lowres.stl" />
         </geometry>
       </collision>

File: stowing/src/stowing_driver/urdf/gripper.urdf.xacro (robot description, xacro)
@@ -10,10 +10,10 @@
 			<visual>
 		        <geometry>
-		        	<mesh filename="package://stowing_driver/scripts/gripper.dae" scale="0.001 0.001 0.001" />
+		        	<mesh filename="package://stowing_driver/meshes/gripper.dae" scale="0.001 0.001 0.001" />
 		        </geometry>
 	  		</visual>
 	    	<collision>
 	    		<geometry>
-	          		<mesh filename="package://stowing_driver/scripts/gripper.dae" scale="0.001 0.001 0.001" />
+	          		<mesh filename="package://stowing_driver/meshes/gripper.dae" scale="0.001 0.001 0.001" />
 	        	</geometry>
 	      	</collision>
@@ -33,10 +33,10 @@
 			<visual>
 		        <geometry>
-		        	<mesh filename="package://stowing_driver/scripts/realsense200.dae" scale="0.001 0.001 0.001" />
+		        	<mesh filename="package://stowing_driver/meshes/realsense200.dae" scale="0.001 0.001 0.001" />
 		        </geometry>
 	  		</visual>
 	    	<collision>
 	    		<geometry>
-	          		<mesh filename="package://stowing_driver/scripts/realsense200.dae" scale="0.001 0.001 0.001" />
+	          		<mesh filename="package://stowing_driver/meshes/realsense200.dae" scale="0.001 0.001 0.001" />
 	        	</geometry>
 	      	</collision>
