Commit message: Further work on state machine

File: stowing/src/stowing_driver/urdf/new_shelf.urdf.xacro (robot description, xacro)
@@ -14,5 +14,5 @@
         <origin xyz="${X} ${Y} ${Z}" rpy="${roll} ${pitch} ${yaw}"/>
         <geometry>
-           <mesh filename="package://stowing_driver/meshes/shelf_9_bin.dae" scale="0.001 0.001 0.001" />
+           <mesh filename="package://stowing_driver/meshes/billy_combined.dae" scale="0.001 0.001 0.001" />
         </geometry>
       </visual>
@@ -20,5 +20,5 @@
         <origin xyz="${X} ${Y} ${Z}" rpy="${roll} ${pitch} ${yaw}"/>
         <geometry>
-           <mesh filename="package://stowing_driver/meshes/shelf_9_bin.dae" scale="0.001 0.001 0.001" />
+           <mesh filename="package://stowing_driver/meshes/billy_combined.dae" scale="0.001 0.001 0.001" />
         </geometry>
       </collision>

File: stowing/src/stowing_driver/urdf/tote_1.urdf.xacro (robot description, xacro)
@@ -1,5 +1,5 @@
 <?xml version="1.0"?>
 <robot xmlns:xacro="http://www.ros.org/wiki/xacro" name="spawn_tote_1">
-	<xacro:tote_1 X="0.25" Y="0.4" Z="0.5" roll="1.571" pitch="0.0" yaw="0.0"/>
+	<xacro:tote_1 X="0.10" Y="0.4" Z="0.5" roll="1.571" pitch="0.0" yaw="0.0"/>
 	<xacro:macro name="tote_1" params="X Y Z roll pitch yaw">
 		<link name="world" />

File: stowing/src/stowing_driver/urdf/tote_amnesty.urdf.xacro (robot description, xacro)
@@ -1,5 +1,5 @@
 <?xml version="1.0"?>
 <robot xmlns:xacro="http://www.ros.org/wiki/xacro" name="spawn_tote_amnesty">
-	<xacro:tote_amnesty X="0.25" Y="0.0" Z="0.5" roll="1.571" pitch="0.0" yaw="0.0"/>
+	<xacro:tote_amnesty X="0.10" Y="0.0" Z="0.5" roll="1.571" pitch="0.0" yaw="0.0"/>
 	<xacro:macro name="tote_amnesty" params="X Y Z roll pitch yaw">
 		<link name="world" />
